Commit message: update repo

File: urdf/udacity_bot.xacro (robot description, xacro)
@@ -1,5 +1,5 @@
 <?xml version='1.0'?>
 <robot name="udacity_my_robot" xmlns:xacro="http://www.ros.org/wiki/xacro">
-  <xacro:include filename="$(find udacity_my_robot)/urdf/udacity_bot.gazebo"/>
+  <xacro:include filename="$(find slam_project)/urdf/udacity_bot.gazebo"/>
   <link name="robot_footprint"></link>
   <joint name="robot_footprint_joint" type="fixed">
@@ -211,5 +211,5 @@
     <visual name='hokuyo_visual'>
       <geometry>
-          <mesh filename="package://udacity_my_robot/meshes/hokuyo.dae"/>
+          <mesh filename="package://slam_project/meshes/hokuyo.dae"/>
       </geometry>
     </visual>

Commit message: mapping shows correct orientation now

File: urdf/udacity_bot.xacro (robot description, xacro)
@@ -11,5 +11,5 @@
     <pose>0 0 0.2 1 0 0</pose>
     <inertial>
-      <mass value="15.0"/>
+      <mass value="20.0"/>
       <origin xyz="0.0 0 0.15" rpy=" 0 0 0"/>
       <inertia
@@ -94,5 +94,5 @@
     <axis xyz="0 1 0" rpy="0 0 0"/>
     <limit effort="10000" velocity="1000"/>
-    <joint_properties damping="1.0" friction="1.5"/>
+    <joint_properties damping="1.0" friction="2.0"/>
   </joint>
 <!-- RIGHT BACK WHEEL -->
@@ -158,5 +158,5 @@
     <axis xyz="0 1 0" rpy="0 0 0"/>
     <limit effort="10000" velocity="1000"/>
-    <joint_properties damping="1.0" friction="1.5"/>
+    <joint_properties damping="1.0" friction="2.0"/>
   </joint>
   <!-- CAMERA -->
@@ -192,6 +192,5 @@
     <joint_properties damping="1.0" friction="1.0"/>
   </joint>
-  <!-- LASER RANGE FINDER-->
-  <link name="hokuyo">
+  <link name="camera_optical">
     <inertial>
       <mass value="0.1"/>
@@ -203,4 +202,36 @@
       />
     </inertial>
+    <collision name='camera_collision'>
+      <origin xyz="0 0 0" rpy=" 0 0 0"/>
+      <geometry>
+        <box size="0.05 0.05 0.05"/>
+      </geometry>
+    </collision>
+    <visual name='camera_visual'>
+      <origin xyz="0 0 0" rpy="0 0 0"/>
+      <geometry>
+        <box size="0.02 0.02 0.02"/>
+      </geometry>
+    </visual>
+  </link>
+  <joint type="fixed" name="camera_optical_joint">
+    <origin xyz="0.22 0 0.18" rpy="-1.57 0 -1.57"/>
+    <child link="camera_optical"/>
+    <parent link="chassis"/>
+    <axis xyz="0 0 0" rpy="0 0 0"/>
+    <limit effort="10000" velocity="1000"/>
+    <joint_properties damping="1.0" friction="1.0"/>
+  </joint>
+  <!-- LASER RANGE FINDER-->
+  <link name="hokuyo">
+    <inertial>
+      <mass value="0.1"/>
+      <origin xyz="0 0 0" rpy=" 0 0 0"/>
+      <inertia
+          ixx="1e-6" ixy="0" ixz="0"
+          iyy="1e-6" iyz="0"
+          izz="1e-6"
+      />
+    </inertial>
     <collision name='hokuyo_collision'>
       <origin xyz="0 0 0" rpy=" 0 0 0"/>

Commit message: change robot design for ease of control

File: urdf/udacity_bot.xacro (robot description, xacro)
@@ -11,5 +11,5 @@
     <pose>0 0 0.2 1 0 0</pose>
     <inertial>
-      <mass value="20.0"/>
+      <mass value="10.0"/>
       <origin xyz="0.0 0 0.15" rpy=" 0 0 0"/>
       <inertia
@@ -46,5 +46,5 @@
       <origin xyz="0 0 0" rpy=" 0 1.5707 1.5707"/>
       <geometry>
-        <cylinder length="0.07" radius="0.08"/>
+        <cylinder length="0.03" radius="0.08"/>
       </geometry>
     </collision>
@@ -52,5 +52,5 @@
       <origin xyz="0 0 0" rpy=" 0 1.5707 1.5707"/>
       <geometry>
-        <cylinder length="0.07" radius="0.08"/>
+        <cylinder length="0.03" radius="0.08"/>
       </geometry>
     </visual>
@@ -78,5 +78,5 @@
       <origin xyz="0 0 0" rpy=" 0 1.5707 1.5707"/>
       <geometry>
-        <cylinder length="0.07" radius="0.08"/>
+        <cylinder length="0.03" radius="0.08"/>
       </geometry>
     </collision>
@@ -84,5 +84,5 @@
       <origin xyz="0 0 0" rpy=" 0 1.5707 1.5707"/>
       <geometry>
-        <cylinder length="0.07" radius="0.08"/>
+        <cylinder length="0.03" radius="0.08"/>
       </geometry>
     </visual>
@@ -110,5 +110,5 @@
       <origin xyz="0 0 0" rpy=" 0 1.5707 1.5707"/>
       <geometry>
-        <cylinder length="0.07" radius="0.08"/>
+        <cylinder length="0.03" radius="0.08"/>
       </geometry>
     </collision>
@@ -116,5 +116,5 @@
       <origin xyz="0 0 0" rpy=" 0 1.5707 1.5707"/>
       <geometry>
-        <cylinder length="0.07" radius="0.08"/>
+        <cylinder length="0.03" radius="0.08"/>
       </geometry>
     </visual>
@@ -142,5 +142,5 @@
       <origin xyz="0 0 0" rpy=" 0 1.5707 1.5707"/>
       <geometry>
-        <cylinder length="0.07" radius="0.08"/>
+        <cylinder length="0.03" radius="0.08"/>
       </geometry>
     </collision>
@@ -148,5 +148,5 @@
       <origin xyz="0 0 0" rpy=" 0 1.5707 1.5707"/>
       <geometry>
-        <cylinder length="0.07" radius="0.08"/>
+        <cylinder length="0.03" radius="0.08"/>
       </geometry>
     </visual>

Commit message: fix robot pose

File: urdf/udacity_bot.xacro (robot description, xacro)
@@ -12,5 +12,5 @@
     <inertial>
       <mass value="10.0"/>
-      <origin xyz="0.0 0 0.15" rpy=" 0 0 0"/>
+      <origin xyz="0.0 0 0.1" rpy=" 0 0 0"/>
       <inertia
           ixx="0.1" ixy="0" ixz="0"
@@ -20,5 +20,5 @@
     </inertial>
     <collision name='collision'>
-      <origin xyz="0 0 0.15" rpy=" 0 0 0"/>
+      <origin xyz="0 0 0.1" rpy=" 0 0 0"/>
       <geometry>
         <box size=".35 .3 .11"/>
@@ -26,7 +26,7 @@
     </collision>
     <visual name='chassis_visual'>
-      <origin xyz="0 0 0.15" rpy=" 0 0 0"/>
-      <geometry>
-        <box size=".4 .3 .11"/>
+      <origin xyz="0 0 0.1" rpy=" 0 0 0"/>
+      <geometry>
+        <box size=".35 .3 .11"/>
       </geometry>
     </visual>
@@ -57,5 +57,5 @@
   </link>
   <joint type="continuous" name="left_back_wheel_hinge">
-    <origin xyz="0.15 0.19 0" rpy="0 0 0"/>
+    <origin xyz="0.15 0.164 0" rpy="0 0 0"/>
     <child link="left_back_wheel"/>
     <parent link="chassis"/>
@@ -89,5 +89,5 @@
   </link>
   <joint type="continuous" name="left_front_wheel_hinge">
-    <origin xyz="-0.15 0.19 0" rpy="0 0 0"/>
+    <origin xyz="-0.15 0.164 0" rpy="0 0 0"/>
     <child link="left_front_wheel"/>
     <parent link="chassis"/>
@@ -121,5 +121,5 @@
   </link>
   <joint type="continuous" name="right_back_wheel_hinge">
-    <origin xyz="0.15 -0.19 0" rpy="0 0 0"/>
+    <origin xyz="0.15 -0.164 0" rpy="0 0 0"/>
     <child link="right_back_wheel"/>
     <parent link="chassis"/>
@@ -153,5 +153,5 @@
   </link>
   <joint type="continuous" name="right_front_wheel_hinge">
-    <origin xyz="-0.15 -0.19 0" rpy="0 0 0"/>
+    <origin xyz="-0.15 -0.164 0" rpy="0 0 0"/>
     <child link="right_front_wheel"/>
     <parent link="chassis"/>
@@ -185,5 +185,5 @@
   </link>
   <joint type="fixed" name="camera_joint">
-    <origin xyz="0.22 0 0.18" rpy="0 0 0"/>
+    <origin xyz="0.18 0 0.16" rpy="0 0 0"/>
     <child link="camera"/>
     <parent link="chassis"/>
@@ -216,5 +216,5 @@
   </link>
   <joint type="fixed" name="camera_optical_joint">
-    <origin xyz="0.22 0 0.18" rpy="-1.57 0 -1.57"/>
+    <origin xyz="0.18 0 0.16" rpy="-1.57 0 -1.57"/>
     <child link="camera_optical"/>
     <parent link="chassis"/>
@@ -247,5 +247,5 @@
   </link>
   <joint type="fixed" name="hokuyo_joint">
-    <origin xyz="-0.07 0 0.3" rpy="0 0 0"/>
+    <origin xyz="-0.07 0 0.17" rpy="0 0 0"/>
     <child link="hokuyo"/>
     <parent link="chassis"/>
